Commit message: grasp fixedgit add .

File: src/urdf/queenie copy 4.xacro (robot description, xacro)
@@ -15,7 +15,7 @@
       <origin xyz="${x} ${y} ${z}" rpy="${r} ${p} ${yaw}"/>
       <mass value="${mass}" />
-      <inertia ixx="${(1/12) * mass * (y_length*y_length + z_length*z_length) * 10}" ixy="0.0" ixz="0.0"
-               iyy="${(1/12) * mass * (x_length*x_length + z_length*z_length) * 10}" iyz="0.0"
-               izz="${(1/12) * mass * (x_length*x_length + y_length*y_length) * 10}" />
+      <inertia ixx="${(1/12) * mass * (y_length*y_length + z_length*z_length) * 100}" ixy="0.0" ixz="0.0"
+               iyy="${(1/12) * mass * (x_length*x_length + z_length*z_length) * 100}" iyz="0.0"
+               izz="${(1/12) * mass * (x_length*x_length + y_length*y_length) * 100}" />
     </inertial>
   </xacro:macro>
@@ -24,7 +24,7 @@
       <origin xyz="${x} ${y} ${z}" rpy="${r} ${p} ${yaw}"/>
       <mass value="${mass}" />
-      <inertia ixx="${(1/12) * mass * (3*radius*radius + height*height) * 10}" ixy="0.0" ixz="0.0"
-               iyy="${(1/12) * mass * (3*radius*radius + height*height) * 10}" iyz="0.0"
-               izz="${(1/2) * mass * radius*radius * 10}" />
+      <inertia ixx="${(1/12) * mass * (3*radius*radius + height*height) * 100}" ixy="0.0" ixz="0.0"
+               iyy="${(1/12) * mass * (3*radius*radius + height*height) * 100}" iyz="0.0"
+               izz="${(1/2) * mass * radius*radius * 100}" />
     </inertial>
   </xacro:macro>
@@ -78,5 +78,5 @@
     <parent link="chassis"/>
     <child link="gripper_pole"/>
-    <limit effort="1000.0" lower="-0.13" upper="0" velocity="0.05"/>
+    <limit effort="1000.0" lower="-0.13" upper="0" velocity="0.5"/>
     <origin rpy="0 0 0" xyz="0.25 0 0"/>
   </joint>
@@ -100,5 +100,5 @@
     <child link="gripper_pole_vertical"/>
     <!-- <limit effort="1000.0" lower="-0.13" upper="0" velocity="0.5"/> -->
-    <origin rpy="0 0 0" xyz="0.225 0 0"/>
+    <origin rpy="0 0 0" xyz="0.2 0 0"/>
   </joint>
   <link name="gripper_pole_vertical">
@@ -120,5 +120,5 @@
     <parent link="gripper_pole_vertical"/>
     <child link="palm"/>
-    <limit effort="1000.0" lower="0" upper="0.9" velocity="0.05"/>
+    <limit effort="1000.0" lower="0" upper="0.09" velocity="0.5"/>
     <origin rpy="0 0 0" xyz="0.01 0 0"/>
     <axis xyz="0 0 1"/>
@@ -127,5 +127,5 @@
       <collision name="collision">
         <geometry>
-          <box size="0.05 0.25 0.05"/>
+          <box size="0.05 0.1 0.05"/>
         </geometry>
         <origin rpy="0 0 0 " xyz="0.025 0 0"/>
@@ -133,53 +133,97 @@
       <visual name="visual">
         <geometry>
-          <box size="0.05 0.25 0.05"/>
+          <box size="0.05 0.1 0.05"/>
         </geometry>
         <origin rpy="0 0 0 " xyz="0.025 0 0"/>
       </visual>
-      <xacro:default_inertial_cuboid mass="0.01" x_length="0.05" y_length="0.25" z_length="0.05" x="0.025" y="0" z="0"/>
-  </link>
-  <joint name="palm_left_finger" type="prismatic">
+      <xacro:default_inertial_cuboid mass="0.01" x_length="0.05" y_length="0.1" z_length="0.05" x="0.025" y="0" z="0"/>
+  </link>
+  <joint name="palm_left_finger" type="revolute">
     <child link="left_finger"/>
     <parent link="palm"/>
-    <limit effort="1000.0" lower="0" upper="0.1" velocity="0.5"/>
-    <origin rpy="0 0 0" xyz="0.125 0.025 0"/>
-    <axis xyz="0 1 0"/>
+    <limit effort="1000.0" lower="-0.4" upper="0.4" velocity="0.5"/>
+    <origin rpy="0 0 ${-pi/4}" xyz="0.025 0.05 0"/>
+    <axis xyz="0 0 -1"/>
   </joint>
   <link name="left_finger">
     <collision name="collision">
       <geometry>
-        <box size="0.15 0.05 0.05"/>
-      </geometry>
-      <origin xyz="0 0 0" rpy="0 0 0 "/>
+        <box size="0.05 0.15 0.05"/>
+      </geometry>
+      <origin xyz="0 0.075 0" rpy="0 0 0 "/>
     </collision>
     <visual name="visual">
       <geometry>
-        <box size="0.15 0.05 0.05"/>
-      </geometry>
-      <origin xyz="0 0 0" rpy="0 0 0 "/>
-    </visual>
-    <xacro:default_inertial_cuboid mass="0.02" x_length="0.15" y_length="0.05" z_length="0.05" x="0" y="0" z="0"/>
-  </link>
-  <joint name="palm_right_finger" type="prismatic">
+        <box size="0.05 0.15 0.05"/>
+      </geometry>
+      <origin xyz="0 0.075 0" rpy="0 0 0 "/>
+    </visual>
+    <xacro:default_inertial_cuboid mass="0.02" x_length="0.05" y_length="0.15" z_length="0.05" x="0" y="0.075" z="0"/>
+  </link>
+  <joint name="left_finger_to_tip" type="revolute">
+    <child link="left_finger_tip"/>
+    <parent link="left_finger"/>
+    <limit effort="1000.0" lower="-0.4" upper="0.4" velocity="0.5"/>
+    <origin rpy="0 0 ${-pi/2}" xyz="0 0.15 0"/>
+    <axis xyz="0 0 -1"/>
+  </joint>
+  <link name="left_finger_tip">
+      <collision>
+          <geometry>
+              <box size="0.05 0.1 0.05"/>
+          </geometry>
+          <origin rpy="0 0 0" xyz="0 0.05 0"/>
+      </collision>
+      <visual name="visual">
+          <geometry>
+              <box size="0.05 0.1 0.05"/>
+          </geometry>
+          <origin rpy="0 0 0" xyz="0 0.05 0"/>
+      </visual>
+      <xacro:default_inertial_cuboid mass="0.01" x_length="0.05" y_length="0.1" z_length="0.05" x="0" y="0.05" z="0"/>
+  </link>
+  <joint name="palm_right_finger" type="revolute">
     <child link="right_finger"/>
     <parent link="palm"/>
-    <limit effort="1000.0" lower="0" upper="0.1" velocity="0.5"/>
-    <origin rpy="0 0 0" xyz="0.125 -0.025 0"/>
-    <axis xyz="0 -1 0"/>
+    <limit effort="1000.0" lower="-0.4" upper="0.4" velocity="0.5"/>
+    <origin rpy="0 0 ${pi/4}" xyz="0.025 -0.05 0"/>
+    <axis xyz="0 0 1"/>
   </joint>
   <link name="right_finger">
     <collision name="collision">
       <geometry>
-        <box size="0.15 0.05 0.05"/>
-      </geometry>
-      <origin xyz="0 0 0" rpy="0 0 0 "/>
+        <box size="0.05 0.15 0.05"/>
+      </geometry>
+      <origin xyz="0 -0.075 0" rpy="0 0 0 "/>
     </collision>
     <visual name="visual">
       <geometry>
-        <box size="0.15 0.05 0.05"/>
-      </geometry>
-      <origin xyz="0 0 0" rpy="0 0 0 "/>
-    </visual>
-    <xacro:default_inertial_cuboid mass="0.02" x_length="0.15" y_length="0.05" z_length="0.05" x="0" y="0" z="0"/>
+        <box size="0.05 0.15 0.05"/>
+      </geometry>
+      <origin xyz="0 -0.075 0" rpy="0 0 0 "/>
+    </visual>
+    <xacro:default_inertial_cuboid mass="0.02" x_length="0.05" y_length="0.15" z_length="0.05" x="0" y="-0.075" z="0"/>
+  </link>
+  <joint name="right_finger_to_tip" type="revolute">
+    <child link="right_finger_tip"/>
+    <parent link="right_finger"/>
+    <limit effort="1000.0" lower="-0.4" upper="0.4" velocity="0.5"/>
+    <origin rpy="0 0 ${pi/2}" xyz="0 -0.15 0"/>
+    <axis xyz="0 0 1"/>
+  </joint>
+  <link name="right_finger_tip">
+      <collision>
+          <geometry>
+              <box size="0.05 0.1 0.05"/>
+          </geometry>
+          <origin rpy="0 0 0" xyz="0 -0.05 0"/>
+      </collision>
+      <visual name="visual">
+          <geometry>
+              <box size="0.05 0.1 0.05"/>
+          </geometry>
+          <origin rpy="0 0 0" xyz="0 -0.05 0"/>
+      </visual>
+      <xacro:default_inertial_cuboid mass="0.01" x_length="0.05" y_length="0.1" z_length="0.05" x="0" y="-0.05" z="0"/>
   </link>
   <joint type="continuous" name="left_wheel_hinge">
