Commit message: updted move

File: src/urdf/queenie.xacro (robot description, xacro)
@@ -188,5 +188,5 @@
     <child link="left_wheel" />
     <axis xyz="0 1 0" rpy="0 0 0" />
-    <limit effort="10000" velocity="1000" />
+    <limit effort="1000000" velocity="1000" />
     <dynamics damping="1.0" friction="1.0" />
   </joint>
@@ -211,5 +211,5 @@
     <child link="right_wheel" />
     <axis xyz="0 1 0" rpy="0 0 0" />
-    <limit effort="10000" velocity="1000" />
+    <limit effort="1000000" velocity="1000" />
     <dynamics damping="1.0" friction="1.0" />
   </joint>

Commit message: fixed grasp again by adding higher inertia values

File: src/urdf/queenie.xacro (robot description, xacro)
@@ -15,7 +15,7 @@
       <origin xyz="${x} ${y} ${z}" rpy="${r} ${p} ${yaw}"/>
       <mass value="${mass}" />
-      <inertia ixx="${(1/12) * mass * (y_length*y_length + z_length*z_length) * 10}" ixy="0.0" ixz="0.0"
-               iyy="${(1/12) * mass * (x_length*x_length + z_length*z_length) * 10}" iyz="0.0"
-               izz="${(1/12) * mass * (x_length*x_length + y_length*y_length) * 10}" />
+      <inertia ixx="${(1/12) * mass * (y_length*y_length + z_length*z_length) * 100}" ixy="0.0" ixz="0.0"
+               iyy="${(1/12) * mass * (x_length*x_length + z_length*z_length) * 100}" iyz="0.0"
+               izz="${(1/12) * mass * (x_length*x_length + y_length*y_length) * 100}" />
     </inertial>
   </xacro:macro>
@@ -24,6 +24,6 @@
       <origin xyz="${x} ${y} ${z}" rpy="${r} ${p} ${yaw}"/>
       <mass value="${mass}" />
-      <inertia ixx="${(1/12) * mass * (3*radius*radius + height*height) * 10}" ixy="0.0" ixz="0.0"
-               iyy="${(1/12) * mass * (3*radius*radius + height*height) * 10}" iyz="0.0"
+      <inertia ixx="${(1/12) * mass * (3*radius*radius + height*height) * 100}" ixy="0.0" ixz="0.0"
+               iyy="${(1/12) * mass * (3*radius*radius + height*height) * 100}" iyz="0.0"
                izz="${(1/2) * mass * radius*radius * 10}" />
     </inertial>
@@ -75,8 +75,8 @@
     </visual>
   </link>
-  <joint name="gripper_extension" type="prismatic">
+  <joint name="gripper_extension" type="fixed">
     <parent link="chassis"/>
     <child link="gripper_pole"/>
-    <limit effort="1000.0" lower="-0.13" upper="0" velocity="0.05"/>
+    <!-- <limit effort="1000.0" lower="-0.13" upper="0" velocity="0.05"/> -->
     <origin rpy="0 0 0" xyz="0.25 0 0"/>
   </joint>

Commit message: basic pick n place implemented

File: src/urdf/queenie.xacro (robot description, xacro)
@@ -250,11 +250,11 @@
       </visual>
     </link>
-  <!-- <joint name="hokuyo_joint" type="fixed">
+  <joint name="hokuyo_joint" type="fixed">
     <origin xyz="0.2 0 0.2" rpy="0 0 0" />
     <parent link="chassis"/>
     <child link="hokuyo" />
     <axis xyz="0 1 0"/>
-  </joint> -->
-  <!-- <link name="hokuyo">
+  </joint>
+  <link name="hokuyo">
     <inertial>
       <mass value="1e-5"/>
@@ -278,4 +278,4 @@
       </geometry>
     </visual>
-  </link> -->
+  </link>
 </robot>

Commit message: latest changes

File: src/urdf/queenie.xacro (robot description, xacro)
@@ -275,5 +275,5 @@
       <origin xyz="0 0 0" rpy="0 0 0"/>
       <geometry>
-        <mesh filename="package://queenie/meshes/hokuyo.dae"/>
+        <mesh filename="package://queenie/src/meshes/hokuyo.dae"/>
       </geometry>
     </visual>

Commit message: latest changes

File: src/urdf/queenie.xacro (robot description, xacro)
@@ -103,10 +103,10 @@
   </joint>
   <link name="gripper_pole_vertical">
-    <visual>
+    <!-- <visual>
       <geometry>
         <box size="0.05 0.05 0.1"/>
       </geometry>
       <origin rpy="0 0 0 " xyz="0 0 0.05"/>
-    </visual>
+    </visual> -->
     <collision>
       <geometry>
@@ -250,4 +250,10 @@
       </visual>
     </link>
+    <joint name="camera_optical_joint" type="fixed">
+      <parent link="camera"/>
+      <child link="camera_optical"/>
+      <origin xyz="0.0 0.0 0.0" rpy="${-pi/2} 0.0 ${-pi/2}"/>
+    </joint>
+    <link name="camera_optical"></link>
   <joint name="hokuyo_joint" type="fixed">
     <origin xyz="0.2 0 0.2" rpy="0 0 0" />

Commit message: latest changes before new year

File: src/urdf/queenie.xacro (robot description, xacro)
@@ -233,5 +233,5 @@
     <parent link="chassis"/>
     <child link="camera" />
-    <axis xyz="0 1 0"/>
+    <axis xyz="0 0 1"/>
   </joint>
   <link name="camera">

Commit message: latest changes

File: src/urdf/queenie.xacro (robot description, xacro)
@@ -15,7 +15,7 @@
       <origin xyz="${x} ${y} ${z}" rpy="${r} ${p} ${yaw}"/>
       <mass value="${mass}" />
-      <inertia ixx="${(1/12) * mass * (y_length*y_length + z_length*z_length) * 100}" ixy="0.0" ixz="0.0"
-               iyy="${(1/12) * mass * (x_length*x_length + z_length*z_length) * 100}" iyz="0.0"
-               izz="${(1/12) * mass * (x_length*x_length + y_length*y_length) * 100}" />
+      <inertia ixx="${(1/12) * mass * (y_length*y_length + z_length*z_length) * 10}" ixy="0.0" ixz="0.0"
+               iyy="${(1/12) * mass * (x_length*x_length + z_length*z_length) * 10}" iyz="0.0"
+               izz="${(1/12) * mass * (x_length*x_length + y_length*y_length) * 10}" />
     </inertial>
   </xacro:macro>
@@ -24,6 +24,6 @@
       <origin xyz="${x} ${y} ${z}" rpy="${r} ${p} ${yaw}"/>
       <mass value="${mass}" />
-      <inertia ixx="${(1/12) * mass * (3*radius*radius + height*height) * 100}" ixy="0.0" ixz="0.0"
-               iyy="${(1/12) * mass * (3*radius*radius + height*height) * 100}" iyz="0.0"
+      <inertia ixx="${(1/12) * mass * (3*radius*radius + height*height) * 10}" ixy="0.0" ixz="0.0"
+               iyy="${(1/12) * mass * (3*radius*radius + height*height) * 10}" iyz="0.0"
                izz="${(1/2) * mass * radius*radius * 10}" />
     </inertial>
@@ -36,6 +36,5 @@
   </joint>
   <link name='chassis'>
-    <!-- <pose>0 0 0.1 0 0 0</pose> -->
-    <xacro:default_inertial_cylinder mass="5" radius="0.25" height="0.2" x="0" y="0" z="0.05" r="0" p="0" yaw="0"/>
+    <xacro:default_inertial_cylinder mass="15" radius="0.25" height="0.2" x="0" y="0" z="0.05" r="0" p="0" yaw="0"/>
     <collision name='collision'>
       <origin xyz="0 0 0.05" rpy=" 0 0 0"/>
@@ -94,5 +93,5 @@
       <origin rpy="0 ${0} 0 " xyz="0.1 0 0"/>
     </collision>
-    <xacro:default_inertial_cuboid mass="0.01" x_length="0.2" y_length="0.05" z_length="0.05" x="0.1" y="0" z="0" r="0" p="0" yaw="0"/>
+    <xacro:default_inertial_cuboid mass="0.5" x_length="0.2" y_length="0.05" z_length="0.05" x="0.1" y="0" z="0" r="0" p="0" yaw="0"/>
   </link>
   <joint name="gripper_extension_vertical" type="fixed">
@@ -103,10 +102,10 @@
   </joint>
   <link name="gripper_pole_vertical">
-    <!-- <visual>
+    <visual>
       <geometry>
         <box size="0.05 0.05 0.1"/>
       </geometry>
       <origin rpy="0 0 0 " xyz="0 0 0.05"/>
-    </visual> -->
+    </visual>
     <collision>
       <geometry>
@@ -115,5 +114,5 @@
       <origin rpy="0 0 0 " xyz="0 0 0.05"/>
     </collision>
-    <xacro:default_inertial_cuboid mass="0.01" x_length="0.05" y_length="0.05" z_length="0.1" x="0" y="0" z="0.05" r="0" p="0" yaw="0"/>
+    <xacro:default_inertial_cuboid mass="0.3" x_length="0.05" y_length="0.05" z_length="0.1" x="0" y="0" z="0.05" r="0" p="0" yaw="0"/>
   </link>
   <joint name="palm_riser" type="prismatic">
@@ -121,5 +120,5 @@
     <child link="palm"/>
     <limit effort="1000.0" lower="0" upper="0.9" velocity="0.05"/>
-    <origin rpy="0 0 0" xyz="0.01 0 0"/>
+    <origin rpy="0 0 0" xyz="0.025 0 0"/>
     <axis xyz="0 0 1"/>
   </joint>
@@ -137,5 +136,5 @@
         <origin rpy="0 0 0 " xyz="0.025 0 0"/>
       </visual>
-      <xacro:default_inertial_cuboid mass="0.01" x_length="0.05" y_length="0.25" z_length="0.05" x="0.025" y="0" z="0"/>
+      <xacro:default_inertial_cuboid mass="0.3" x_length="0.05" y_length="0.25" z_length="0.05" x="0.025" y="0" z="0"/>
   </link>
   <joint name="palm_left_finger" type="prismatic">
@@ -159,5 +158,5 @@
       <origin xyz="0 0 0" rpy="0 0 0 "/>
     </visual>
-    <xacro:default_inertial_cuboid mass="0.02" x_length="0.15" y_length="0.05" z_length="0.05" x="0" y="0" z="0"/>
+    <xacro:default_inertial_cuboid mass="0.3" x_length="0.15" y_length="0.05" z_length="0.05" x="0" y="0" z="0"/>
   </link>
   <joint name="palm_right_finger" type="prismatic">
@@ -181,5 +180,5 @@
       <origin xyz="0 0 0" rpy="0 0 0 "/>
     </visual>
-    <xacro:default_inertial_cuboid mass="0.02" x_length="0.15" y_length="0.05" z_length="0.05" x="0" y="0" z="0"/>
+    <xacro:default_inertial_cuboid mass="0.3" x_length="0.15" y_length="0.05" z_length="0.05" x="0" y="0" z="0"/>
   </link>
   <joint type="continuous" name="left_wheel_hinge">

Commit message: reasonably good grasp acheived

File: src/urdf/queenie.xacro (robot description, xacro)
@@ -78,20 +78,20 @@
     <child link="gripper_pole"/>
     <!-- <limit effort="1000.0" lower="-0.13" upper="0" velocity="0.05"/> -->
-    <origin rpy="0 0 0" xyz="0.25 0 0"/>
+    <origin rpy="0 0 0" xyz="0.30 0 0"/>
   </joint>
   <link name="gripper_pole">
     <visual>
       <geometry>
-        <box size="0.2 0.05 0.05"/>
-      </geometry>
-      <origin rpy="0 ${0} 0 " xyz="0.1 0 0"/>
-    </visual>
-    <collision>
-      <geometry>
-         <box size="0.2 0.05 0.05"/>
-      </geometry>
-      <origin rpy="0 ${0} 0 " xyz="0.1 0 0"/>
-    </collision>
-    <xacro:default_inertial_cuboid mass="0.5" x_length="0.2" y_length="0.05" z_length="0.05" x="0.1" y="0" z="0" r="0" p="0" yaw="0"/>
+        <box size="0.1 0.05 0.05"/>
+      </geometry>
+      <origin rpy="0 ${0} 0 " xyz="0 0 0"/>
+    </visual>
+    <collision>
+      <geometry>
+         <box size="0.1 0.05 0.05"/>
+      </geometry>
+      <origin rpy="0 ${0} 0 " xyz="0 0 0"/>
+    </collision>
+    <xacro:default_inertial_cuboid mass="0.5" x_length="0.1" y_length="0.05" z_length="0.05" x="0" y="0" z="0" r="0" p="0" yaw="0"/>
   </link>
   <joint name="gripper_extension_vertical" type="fixed">
@@ -99,27 +99,28 @@
     <child link="gripper_pole_vertical"/>
     <!-- <limit effort="1000.0" lower="-0.13" upper="0" velocity="0.5"/> -->
-    <origin rpy="0 0 0" xyz="0.225 0 0"/>
+    <origin rpy="0 0 0" xyz="0.075 0 0"/>
   </joint>
   <link name="gripper_pole_vertical">
     <visual>
       <geometry>
-        <box size="0.05 0.05 0.1"/>
-      </geometry>
-      <origin rpy="0 0 0 " xyz="0 0 0.05"/>
-    </visual>
-    <collision>
-      <geometry>
-        <box size="0.05 0.05 0.1"/>
-      </geometry>
-      <origin rpy="0 0 0 " xyz="0 0 0.05"/>
-    </collision>
-    <xacro:default_inertial_cuboid mass="0.3" x_length="0.05" y_length="0.05" z_length="0.1" x="0" y="0" z="0.05" r="0" p="0" yaw="0"/>
+        <box size="0.05 0.05 0.2"/>
+      </geometry>
+      <origin rpy="0 0 0 " xyz="0 0 0.075"/>
+    </visual>
+    <collision>
+      <geometry>
+        <box size="0.05 0.05 0.2"/>
+      </geometry>
+      <origin rpy="0 0 0 " xyz="0 0 0.075"/>
+    </collision>
+    <xacro:default_inertial_cuboid mass="0.3" x_length="0.05" y_length="0.05" z_length="0.2" x="0" y="0" z="0.075" r="0" p="0" yaw="0"/>
   </link>
   <joint name="palm_riser" type="prismatic">
     <parent link="gripper_pole_vertical"/>
     <child link="palm"/>
-    <limit effort="1000.0" lower="0" upper="0.9" velocity="0.05"/>
+    <limit effort="1000.0" lower="0" upper="0.17" velocity="0.05"/>
     <origin rpy="0 0 0" xyz="0.025 0 0"/>
     <axis xyz="0 0 1"/>
+    <dynamics damping="10.0" friction="1.0" />
   </joint>
   <link name="palm">
@@ -136,5 +137,5 @@
         <origin rpy="0 0 0 " xyz="0.025 0 0"/>
       </visual>
-      <xacro:default_inertial_cuboid mass="0.3" x_length="0.05" y_length="0.25" z_length="0.05" x="0.025" y="0" z="0"/>
+      <xacro:default_inertial_cuboid mass="0.8" x_length="0.05" y_length="0.25" z_length="0.05" x="0.025" y="0" z="0"/>
   </link>
   <joint name="palm_left_finger" type="prismatic">
@@ -144,4 +145,5 @@
     <origin rpy="0 0 0" xyz="0.125 0.025 0"/>
     <axis xyz="0 1 0"/>
+    <dynamics damping="0.1" friction="1.0" />
   </joint>
   <link name="left_finger">
@@ -166,4 +168,5 @@
     <origin rpy="0 0 0" xyz="0.125 -0.025 0"/>
     <axis xyz="0 -1 0"/>
+    <dynamics damping="0.1" friction="1.0" />
   </joint>
   <link name="right_finger">

Commit message: updated robot structure and added contact plugin

File: src/urdf/queenie.xacro (robot description, xacro)
@@ -232,6 +232,6 @@
   </link>
   <joint name="camera_joint" type="fixed">
-    <origin xyz="0.26 0 .075" rpy="0 0 0" />
-    <parent link="chassis"/>
+    <origin xyz="0 0 0.225" rpy="0 0 0" />
+    <parent link="gripper_pole_vertical"/>
     <child link="camera" />
     <axis xyz="0 0 1"/>
@@ -258,5 +258,5 @@
     </joint>
     <link name="camera_optical"></link>
-  <joint name="hokuyo_joint" type="fixed">
+  <!-- <joint name="hokuyo_joint" type="fixed">
     <origin xyz="0.2 0 0.2" rpy="0 0 0" />
     <parent link="chassis"/>
@@ -286,4 +286,4 @@
       </geometry>
     </visual>
-  </link>
+  </link> -->
 </robot>

Commit message: added point counter for explore policy

File: src/urdf/queenie.xacro (robot description, xacro)
@@ -15,7 +15,7 @@
       <origin xyz="${x} ${y} ${z}" rpy="${r} ${p} ${yaw}"/>
       <mass value="${mass}" />
-      <inertia ixx="${(1/12) * mass * (y_length*y_length + z_length*z_length) * 10}" ixy="0.0" ixz="0.0"
-               iyy="${(1/12) * mass * (x_length*x_length + z_length*z_length) * 10}" iyz="0.0"
-               izz="${(1/12) * mass * (x_length*x_length + y_length*y_length) * 10}" />
+      <inertia ixx="${(1/12) * mass * (y_length*y_length + z_length*z_length) * 1}" ixy="0.0" ixz="0.0"
+               iyy="${(1/12) * mass * (x_length*x_length + z_length*z_length) * 1}" iyz="0.0"
+               izz="${(1/12) * mass * (x_length*x_length + y_length*y_length) * 1}" />
     </inertial>
   </xacro:macro>
@@ -24,7 +24,16 @@
       <origin xyz="${x} ${y} ${z}" rpy="${r} ${p} ${yaw}"/>
       <mass value="${mass}" />
-      <inertia ixx="${(1/12) * mass * (3*radius*radius + height*height) * 10}" ixy="0.0" ixz="0.0"
-               iyy="${(1/12) * mass * (3*radius*radius + height*height) * 10}" iyz="0.0"
-               izz="${(1/2) * mass * radius*radius * 10}" />
+      <inertia ixx="${(1/12) * mass * (3*radius*radius + height*height) * 1}" ixy="0.0" ixz="0.0"
+               iyy="${(1/12) * mass * (3*radius*radius + height*height) * 1}" iyz="0.0"
+               izz="${(1/2) * mass * radius*radius * 1}" />
+    </inertial>
+  </xacro:macro>
+  <xacro:macro name="default_inertial_solid_sphere" params="mass radius">
+    <inertial>
+      <origin xyz="0 0 0" rpy="0 0 0"/>
+      <mass value="${mass}" />
+      <inertia ixx="${(2/5) * mass * radius*radius}" ixy="0.0" ixz="0.0"
+               iyy="${(2/5) * mass * radius*radius}" iyz="0.0"
+               izz="${(2/5) * mass * radius*radius}" />
     </inertial>
   </xacro:macro>
@@ -49,5 +58,5 @@
       </geometry>
     </visual>
-    <collision name='back_caster_collision'>
+    <!-- <collision name='back_caster_collision'>
       <origin xyz="-0.15 0 -0.05" rpy=" 0 0 0"/>
       <geometry>
@@ -60,6 +69,6 @@
         <sphere radius="0.05"/>
       </geometry>
-    </visual>
-    <collision name='front_caster_collision'>
+    </visual> -->
+    <!-- <collision name='front_caster_collision'>
       <origin xyz="0.15 0 -0.05" rpy=" 0 0 0"/>
       <geometry>
@@ -69,4 +78,44 @@
     <visual name='front_caster_visual'>
       <origin xyz="0.15 0 -0.05" rpy=" 0 0 0"/>
+      <geometry>
+        <sphere radius="0.05"/>
+      </geometry>
+    </visual> -->
+  </link>
+  <joint name="chassis_front_caster" type="fixed">
+    <parent link="chassis"/>
+    <child link="front_caster"/>
+    <origin xyz="0.15 0 -0.05" rpy="0 0 0"/>
+  </joint>
+  <link name="front_caster">
+  <xacro:default_inertial_solid_sphere mass="0.1" radius="0.0499"/>
+    <collision>
+      <origin xyz="0 0 0" rpy=" 0 0 0"/>
+      <geometry>
+        <sphere radius="0.0499"/>
+      </geometry>
+    </collision>
+    <visual>
+      <origin xyz="0 0 0" rpy=" 0 0 0"/>
+      <geometry>
+        <sphere radius="0.05"/>
+      </geometry>
+    </visual>
+  </link>
+  <joint name="chassis_back_caster" type="fixed">
+    <parent link="chassis"/>
+    <child link="back_caster"/>
+    <origin xyz="-0.15 0 -0.05" rpy="0 0 0"/>
+  </joint>
+  <link name="back_caster">
+  <xacro:default_inertial_solid_sphere mass="0.1" radius="0.0499"/>
+    <collision>
+      <origin xyz="0 0 0" rpy=" 0 0 0"/>
+      <geometry>
+        <sphere radius="0.0499"/>
+      </geometry>
+    </collision>
+    <visual>
+      <origin xyz="0 0 0" rpy=" 0 0 0"/>
       <geometry>
         <sphere radius="0.05"/>
@@ -258,32 +307,3 @@
     </joint>
     <link name="camera_optical"></link>
-  <!-- <joint name="hokuyo_joint" type="fixed">
-    <origin xyz="0.2 0 0.2" rpy="0 0 0" />
-    <parent link="chassis"/>
-    <child link="hokuyo" />
-    <axis xyz="0 1 0"/>
-  </joint>
-  <link name="hokuyo">
-    <inertial>
-      <mass value="1e-5"/>
-      <origin xyz="0 0 0" rpy="0 0 0"/>
-      <inertia
-        ixx="1e-6" ixy="0.0" ixz="0.0"
-        iyy="1e-6" iyz="0.0"
-        izz="1e-6"
-      />
-    </inertial>
-    <collision>
-      <origin xyz="0 0 0" rpy="0 0 0"/>
-      <geometry>
-        <box size="0.1 0.1 0.1"/>
-      </geometry>
-    </collision>
-    <visual>
-      <origin xyz="0 0 0" rpy="0 0 0"/>
-      <geometry>
-        <mesh filename="package://queenie/src/meshes/hokuyo.dae"/>
-      </geometry>
-    </visual>
-  </link> -->
 </robot>

Commit message: left and right finger contact sensor

File: src/urdf/queenie.xacro (robot description, xacro)
@@ -197,5 +197,5 @@
   </joint>
   <link name="left_finger">
-    <collision name="collision">
+    <collision name="left_finger_collision">
       <geometry>
         <box size="0.15 0.05 0.05"/>
@@ -220,5 +220,5 @@
   </joint>
   <link name="right_finger">
-    <collision name="collision">
+    <collision name="right_finger_collision">
       <geometry>
         <box size="0.15 0.05 0.05"/>

Commit message: improved grasp and added color segmentation

File: src/urdf/queenie.xacro (robot description, xacro)
@@ -171,5 +171,5 @@
     <origin rpy="0 0 0" xyz="0.025 0 0"/>
     <axis xyz="0 0 1"/>
-    <dynamics damping="10.0" friction="1.0" />
+    <dynamics damping="1.0" friction="0.1" />
   </joint>
   <link name="palm">

Commit message: added head joint and controllers back in action

File: src/urdf/queenie.xacro (robot description, xacro)
@@ -58,28 +58,4 @@
       </geometry>
     </visual>
-    <!-- <collision name='back_caster_collision'>
-      <origin xyz="-0.15 0 -0.05" rpy=" 0 0 0"/>
-      <geometry>
-        <sphere radius="0.0499"/>
-      </geometry>
-    </collision>
-    <visual name='back_caster_visual'>
-      <origin xyz="-0.15 0 -0.05" rpy=" 0 0 0"/>
-      <geometry>
-        <sphere radius="0.05"/>
-      </geometry>
-    </visual> -->
-    <!-- <collision name='front_caster_collision'>
-      <origin xyz="0.15 0 -0.05" rpy=" 0 0 0"/>
-      <geometry>
-        <sphere radius="0.0499"/>
-      </geometry>
-    </collision>
-    <visual name='front_caster_visual'>
-      <origin xyz="0.15 0 -0.05" rpy=" 0 0 0"/>
-      <geometry>
-        <sphere radius="0.05"/>
-      </geometry>
-    </visual> -->
   </link>
   <joint name="chassis_front_caster" type="fixed">
@@ -144,6 +120,18 @@
     <xacro:default_inertial_cuboid mass="0.5" x_length="0.1" y_length="0.05" z_length="0.05" x="0" y="0" z="0" r="0" p="0" yaw="0"/>
   </link>
-  <joint name="gripper_extension_vertical" type="fixed">
+  <joint name="neck" type="revolute">
     <parent link="gripper_pole"/>
+    <child link="head"/>
+    <limit effort="1000.0" velocity="0.05" lower="${-pi/8}" upper="0.2"/>
+    <origin rpy="0 0 0" xyz="0.0 0 0"/>
+    <axis xyz="0 1 0"/>
+    <dynamics damping="1.0" friction="0.1" />
+  </joint>
+  <link name="head">
+  <xacro:default_inertial_cuboid mass="0.8" x_length="0.01" y_length="0.025" z_length="0.005" x="0.0" y="0" z="0"/>
+  <!-- <visual><geometry><sphere radius=".01"/></geometry></visual> -->
+  </link>
+  <joint name="head_gripper_pole_vertical" type="fixed">
+    <parent link="head"/>
     <child link="gripper_pole_vertical"/>
     <!-- <limit effort="1000.0" lower="-0.13" upper="0" velocity="0.5"/> -->

Commit message: trajectory controller added

File: src/urdf/queenie.xacro (robot description, xacro)
@@ -123,8 +123,8 @@
     <parent link="gripper_pole"/>
     <child link="head"/>
-    <limit effort="1000.0" velocity="0.05" lower="${-pi/8}" upper="0.2"/>
+    <limit effort="1000.0" velocity="0.05" lower="-0.4" upper="0.2"/>
     <origin rpy="0 0 0" xyz="0.0 0 0"/>
     <axis xyz="0 1 0"/>
-    <dynamics damping="1.0" friction="0.1" />
+    <dynamics damping="0.1" friction="0.1" />
   </joint>
   <link name="head">
@@ -159,5 +159,5 @@
     <origin rpy="0 0 0" xyz="0.025 0 0"/>
     <axis xyz="0 0 1"/>
-    <dynamics damping="1.0" friction="0.1" />
+    <dynamics damping="0.1" friction="0.1" />
   </joint>
   <link name="palm">
