Commit message: converted into skid steering

File: src/urdf/queenie.xacro (robot description, xacro)
@@ -59,5 +59,5 @@
     </visual>
   </link>
-  <joint name="chassis_front_caster" type="fixed">
+  <!-- <joint name="chassis_front_caster" type="fixed">
     <parent link="chassis"/>
     <child link="front_caster"/>
@@ -98,5 +98,5 @@
       </geometry>
     </visual>
-  </link>
+  </link> -->
   <joint name="gripper_extension" type="fixed">
     <parent link="chassis"/>
@@ -162,5 +162,5 @@
   </joint>
   <link name="palm">
-      <collision name="collision">
+      <collision name="palm_collision">
         <geometry>
           <box size="0.05 0.25 0.05"/>
@@ -182,5 +182,5 @@
     <origin rpy="0 0 0" xyz="0.125 0.025 0"/>
     <axis xyz="0 1 0"/>
-    <dynamics damping="0.1" friction="1.0" />
+    <dynamics damping="0" friction="0.1" />
   </joint>
   <link name="left_finger">
@@ -205,5 +205,5 @@
     <origin rpy="0 0 0" xyz="0.125 -0.025 0"/>
     <axis xyz="0 -1 0"/>
-    <dynamics damping="0.1" friction="1.0" />
+    <dynamics damping="0" friction="0.1" />
   </joint>
   <link name="right_finger">
@@ -223,5 +223,5 @@
   </link>
   <joint type="continuous" name="left_wheel_hinge">
-    <origin xyz="0 0.30 0" rpy="0 0 0" />
+    <origin xyz="0.15 0.30 0" rpy="0 0 0" />
     <parent link="chassis"/>
     <child link="left_wheel" />
@@ -246,5 +246,5 @@
   </link>
   <joint type="continuous" name="right_wheel_hinge">
-    <origin xyz="0 -0.30 0" rpy="0 0 0" />
+    <origin xyz="0.15 -0.30 0" rpy="0 0 0" />
     <parent link="chassis"/>
     <child link="right_wheel" />
@@ -254,4 +254,50 @@
   </joint>
   <link name="right_wheel">
+    <xacro:default_inertial_cylinder mass="2" radius="0.1" height="0.05" x="0" y="0" z="0" r="0" p="${pi/2}" yaw="${pi/2}"/>
+    <collision>
+      <origin xyz="0 0 0" rpy="0 1.5707 1.5707"/>
+      <geometry>
+        <cylinder radius="0.1" length="0.05"/>
+      </geometry>
+    </collision>
+    <visual>
+      <origin xyz="0 0 0" rpy="0 1.5707 1.5707"/>
+      <geometry>
+        <cylinder radius="0.1" length="0.05"/>
+      </geometry>
+    </visual>
+  </link>
+    <joint type="continuous" name="left_wheel_back_hinge">
+    <origin xyz="-0.15 0.30 0" rpy="0 0 0" />
+    <parent link="chassis"/>
+    <child link="left_wheel_back" />
+    <axis xyz="0 1 0" rpy="0 0 0" />
+    <limit effort="1000000" velocity="1000" />
+    <dynamics damping="1.0" friction="1.0" />
+  </joint>
+  <link name="left_wheel_back">
+    <xacro:default_inertial_cylinder mass="2" radius="0.1" height="0.05" x="0" y="0" z="0" r="0" p="${pi/2}" yaw="${pi/2}"/>
+    <collision>
+      <origin xyz="0 0 0" rpy="0 1.5707 1.5707"/>
+      <geometry>
+        <cylinder radius="0.1" length="0.05"/>
+      </geometry>
+    </collision>
+    <visual>
+      <origin xyz="0 0 0" rpy="0 1.5707 1.5707"/>
+      <geometry>
+        <cylinder radius="0.1" length="0.05"/>
+      </geometry>
+    </visual>
+  </link>
+  <joint type="continuous" name="right_wheel_back_hinge">
+    <origin xyz="-0.15 -0.30 0" rpy="0 0 0" />
+    <parent link="chassis"/>
+    <child link="right_wheel_back" />
+    <axis xyz="0 1 0" rpy="0 0 0" />
+    <limit effort="1000000" velocity="1000" />
+    <dynamics damping="1.0" friction="1.0" />
+  </joint>
+  <link name="right_wheel_back">
     <xacro:default_inertial_cylinder mass="2" radius="0.1" height="0.05" x="0" y="0" z="0" r="0" p="${pi/2}" yaw="${pi/2}"/>
     <collision>

Commit message: reshaped queenie

File: src/urdf/queenie.xacro (robot description, xacro)
@@ -103,5 +103,5 @@
     <child link="gripper_pole"/>
     <!-- <limit effort="1000.0" lower="-0.13" upper="0" velocity="0.05"/> -->
-    <origin rpy="0 0 0" xyz="0.30 0 0"/>
+    <origin rpy="0 0 0" xyz="0.30 0 0.05"/>
   </joint>
   <link name="gripper_pole">
@@ -114,14 +114,14 @@
     <collision>
       <geometry>
-         <box size="0.1 0.05 0.05"/>
+         <box size="0.01 0.05 0.05"/>
       </geometry>
       <origin rpy="0 ${0} 0 " xyz="0 0 0"/>
     </collision>
-    <xacro:default_inertial_cuboid mass="0.5" x_length="0.1" y_length="0.05" z_length="0.05" x="0" y="0" z="0" r="0" p="0" yaw="0"/>
+    <xacro:default_inertial_cuboid mass="0.5" x_length="0.05" y_length="0.05" z_length="0.05" x="0" y="0" z="0" r="0" p="0" yaw="0"/>
   </link>
   <joint name="neck" type="revolute">
     <parent link="gripper_pole"/>
     <child link="head"/>
-    <limit effort="1000.0" velocity="0.05" lower="-0.4" upper="0.2"/>
+    <limit effort="1000.0" velocity="0.05" lower="${-pi/3}" upper="${0.22}"/>
     <origin rpy="0 0 0" xyz="0.0 0 0"/>
     <axis xyz="0 1 0"/>
@@ -132,11 +132,23 @@
   <!-- <visual><geometry><sphere radius=".01"/></geometry></visual> -->
   </link>
+  <joint name="neck_x" type="revolute">
+    <parent link="head"/>
+    <child link="head_x"/>
+    <limit effort="1000.0" velocity="0.05" lower="-0.5" upper="0.5"/>
+    <origin rpy="0 0 0" xyz="0.0 0 0"/>
+    <axis xyz="1 0 0"/>
+    <dynamics damping="0.1" friction="0.1" />
+  </joint>
+  <link name="head_x">
+  <xacro:default_inertial_cuboid mass="0.8" x_length="0.01" y_length="0.025" z_length="0.005" x="0.0" y="0" z="0"/>
+  <!-- <visual><geometry><sphere radius=".01"/></geometry></visual> -->
+  </link>
   <joint name="head_gripper_pole_vertical" type="fixed">
-    <parent link="head"/>
-    <child link="gripper_pole_vertical"/>
+    <parent link="head_x"/>
+    <child link="palm"/>
     <!-- <limit effort="1000.0" lower="-0.13" upper="0" velocity="0.5"/> -->
-    <origin rpy="0 0 0" xyz="0.075 0 0"/>
-  </joint>
-  <link name="gripper_pole_vertical">
+    <origin rpy="0 0 0" xyz="0.05 0 0"/>
+  </joint>
+  <!-- <link name="gripper_pole_vertical">
     <visual>
       <geometry>
@@ -152,6 +164,6 @@
     </collision>
     <xacro:default_inertial_cuboid mass="0.3" x_length="0.05" y_length="0.05" z_length="0.2" x="0" y="0" z="0.075" r="0" p="0" yaw="0"/>
-  </link>
-  <joint name="palm_riser" type="prismatic">
+  </link> -->
+  <!-- <joint name="palm_riser" type="prismatic">
     <parent link="gripper_pole_vertical"/>
     <child link="palm"/>
@@ -160,5 +172,5 @@
     <axis xyz="0 0 1"/>
     <dynamics damping="0.1" friction="0.1" />
-  </joint>
+  </joint> -->
   <link name="palm">
       <collision name="palm_collision">
@@ -315,6 +327,6 @@
   </link>
   <joint name="camera_joint" type="fixed">
-    <origin xyz="0 0 0.225" rpy="0 0 0" />
-    <parent link="gripper_pole_vertical"/>
+    <origin xyz="0.025 0 0.05" rpy="0 0 0" />
+    <parent link="palm"/>
     <child link="camera" />
     <axis xyz="0 0 1"/>
@@ -322,10 +334,10 @@
   <link name="camera">
       <xacro:default_inertial_cuboid mass="0.01" x_length="0.05" y_length="0.05" z_length="0.05" x="0" y="0" z="0"/>
-      <collision>
+      <!-- <collision>
         <origin xyz="0 0 0" rpy="0 0 0"/>
         <geometry>
           <box size="0.05 0.05 0.05"/>
         </geometry>
-      </collision>
+      </collision> -->
       <visual>
         <origin xyz="0 0 0" rpy="0 0 0"/>
